File: sensor_enco.brd (EAGLE design)
At the start: 25 x 25 mm, 26 parts

Commit message: some changes
Parts:
- removed JP3: (no value), pinh2mm2:1X02_2MM
- added C10: (no value), rcl:C0402
- added JP1: (no value), pinh2mm2:1X03_2MM
- added S1: SWITCHMETAL, switchmetal:SWMET
Connections:
- new net N$18: C10.1, JP1.P$3, S1.P$4, S1.P$4@1
- net N$13: now also C10.2, JP1.P$2, S1.P$1, S1.P$1@1; no longer JP3.P$1
- net N$14: now also JP1.P$1; no longer JP3.P$2
Routing:
- net N$18: track 0.00 -> 5.34 mm
- net N$13: track 1.27 -> 3.43 mm, vias 20 -> 21
- net N$14: track 4.19 -> 3.16 mm
- net N$1: track 17.4 -> 18.2 mm
- net N$8: track 15.4 -> 14.8 mm
