File: sensor_enco.sch (EAGLE design)
At the start: 26 parts

Commit message: some changes
Parts:
- removed JP3: (no value), pinh2mm2:PINHD-1X22MM
- added C10: (no value), rcl:C-EUC0402
- added JP1: (no value), pinh2mm2:PINHD-1X32MM
- added S1: SWITCHMETAL, switchmetal:SWITCHMETAL
Connections:
- new net N$18: C10.1, JP1.3, S1.S
- net N$13: now also C10.2, JP1.2, S1.P; no longer JP3.1
- net N$14: now also JP1.1; no longer JP3.2
Changed lines of the file:
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@@
 <part name="R4" library="rcl" library_urn="urn:adsk.eagle:library:334" deviceset="R-EU_" device="R0402" package3d_urn="urn:adsk.eagle:package:23547/3"/>
 <part name="R5" library="rcl" library_urn="urn:adsk.eagle:library:334" deviceset="R-EU_" device="R0402" package3d_urn="urn:adsk.eagle:package:23547/3"/>
-<part name="JP3" library="pinh2mm2" deviceset="PINHD-1X2" device="2MM"/>
 <part name="JP4" library="pinh2mm2" deviceset="PINHD-1X4" device="2MM"/>
 <part name="U$1" library="sensor pad" deviceset="SENSOR_PAD" device="SENSORPAD3"/>
@@
 <part name="U$15" library="sensor pad" deviceset="SENSOR_PAD" device="SENSORPAD3"/>
 <part name="R6" library="rcl" library_urn="urn:adsk.eagle:library:334" deviceset="R-EU_" device="R0402" package3d_urn="urn:adsk.eagle:package:23547/3"/>
+<part name="S1" library="switchmetal" deviceset="SWITCHMETAL" device=""/>
+<part name="JP1" library="pinh2mm2" deviceset="PINHD-1X3" device="2MM"/>
+<part name="C10" library="rcl" library_urn="urn:adsk.eagle:library:334" deviceset="C-EU" device="C0402" package3d_urn="urn:adsk.eagle:package:23626/2"/>
 </parts>
 <sheets>
@@
 <attribute name="NAME" x="67.31" y="21.8186" size="1.778" layer="95"/>
 <attribute name="VALUE" x="67.31" y="17.018" size="1.778" layer="96"/>
-</instance>
-<instance part="JP3" gate="G$1" x="116.84" y="-33.02" smashed="yes">
-<attribute name="NAME" x="110.49" y="-27.305" size="1.778" layer="95"/>
-<attribute name="VALUE" x="110.49" y="-38.1" size="1.778" layer="96"/>
 </instance>
 <instance part="JP4" gate="A" x="134.62" y="-17.78" smashed="yes">
@@
 <attribute name="VALUE" x="10.922" y="-34.29" size="1.778" layer="96" rot="R90"/>
 </instance>
+<instance part="S1" gate="G$1" x="93.98" y="-68.58" smashed="yes">
+<attribute name="NAME" x="90.17" y="-65.405" size="1.778" layer="95" rot="R90"/>
+<attribute name="VALUE" x="92.71" y="-65.405" size="1.778" layer="96" rot="R90"/>
+</instance>
+<instance part="JP1" gate="A" x="116.84" y="-43.18" smashed="yes">
+<attribute name="NAME" x="110.49" y="-37.465" size="1.778" layer="95"/>
+<attribute name="VALUE" x="110.49" y="-50.8" size="1.778" layer="96"/>
+</instance>
+<instance part="C10" gate="G$1" x="104.14" y="-66.04" smashed="yes">
+<attribute name="NAME" x="105.664" y="-65.659" size="1.778" layer="95"/>
+<attribute name="VALUE" x="105.664" y="-70.739" size="1.778" layer="96"/>
+</instance>
 </instances>
 <busses>
@@
 <wire x1="15.24" y1="-50.8" x2="15.24" y2="-60.96" width="0.1524" layer="91"/>
 <wire x1="15.24" y1="-60.96" x2="33.02" y2="-60.96" width="0.1524" layer="91"/>
-<wire x1="33.02" y1="-60.96" x2="78.74" y2="-60.96" width="0.1524" layer="91"/>
-<wire x1="78.74" y1="-60.96" x2="78.74" y2="-30.48" width="0.1524" layer="91"/>
+<wire x1="33.02" y1="-60.96" x2="53.34" y2="-60.96" width="0.1524" layer="91"/>
+<wire x1="53.34" y1="-60.96" x2="78.74" y2="-60.96" width="0.1524" layer="91"/>
 <pinref part="R5" gate="G$1" pin="2"/>
 <wire x1="76.2" y1="20.32" x2="78.74" y2="20.32" width="0.1524" layer="91"/>
-<wire x1="78.74" y1="20.32" x2="78.74" y2="-30.48" width="0.1524" layer="91"/>
+<wire x1="78.74" y1="20.32" x2="78.74" y2="-43.18" width="0.1524" layer="91"/>
 <pinref part="R4" gate="G$1" pin="2"/>
+<wire x1="78.74" y1="-43.18" x2="78.74" y2="-60.96" width="0.1524" layer="91"/>
 <wire x1="76.2" y1="25.4" x2="78.74" y2="25.4" width="0.1524" layer="91"/>
 <wire x1="78.74" y1="25.4" x2="78.74" y2="20.32" width="0.1524" layer="91"/>
@@
 <wire x1="-38.1" y1="-50.8" x2="-30.48" y2="-50.8" width="0.1524" layer="91"/>
 <junction x="-30.48" y="-50.8"/>
-<pinref part="JP3" gate="G$1" pin="1"/>
-<wire x1="114.3" y1="-30.48" x2="78.74" y2="-30.48" width="0.1524" layer="91"/>
-<junction x="78.74" y="-30.48"/>
 <wire x1="7.62" y1="-35.56" x2="7.62" y2="-50.8" width="0.1524" layer="91"/>
 <junction x="7.62" y="-50.8"/>
 <pinref part="R6" gate="G$1" pin="1"/>
+<pinref part="S1" gate="G$1" pin="P"/>
+<wire x1="96.52" y1="-73.66" x2="96.52" y2="-78.74" width="0.1524" layer="91"/>
+<wire x1="96.52" y1="-78.74" x2="53.34" y2="-78.74" width="0.1524" layer="91"/>
+<wire x1="53.34" y1="-78.74" x2="53.34" y2="-60.96" width="0.1524" layer="91"/>
+<junction x="53.34" y="-60.96"/>
+<pinref part="JP1" gate="A" pin="2"/>
+<wire x1="114.3" y1="-43.18" x2="78.74" y2="-43.18" width="0.1524" layer="91"/>
+<junction x="78.74" y="-43.18"/>
+<pinref part="C10" gate="G$1" pin="2"/>
+<wire x1="104.14" y1="-71.12" x2="104.14" y2="-78.74" width="0.1524" layer="91"/>
+<wire x1="104.14" y1="-78.74" x2="96.52" y2="-78.74" width="0.1524" layer="91"/>
+<junction x="96.52" y="-78.74"/>
 </segment>
 </net>
 <net name="N$14" class="0">
 <segment>
-<wire x1="104.14" y1="-38.1" x2="33.02" y2="-38.1" width="0.1524" layer="91"/>
+<wire x1="99.06" y1="-38.1" x2="33.02" y2="-38.1" width="0.1524" layer="91"/>
 <wire x1="33.02" y1="-38.1" x2="12.7" y2="-38.1" width="0.1524" layer="91"/>
 <wire x1="12.7" y1="-38.1" x2="12.7" y2="-30.48" width="0.1524" layer="91"/>
@@
 <wire x1="33.02" y1="-45.72" x2="33.02" y2="-38.1" width="0.1524" layer="91"/>
 <junction x="33.02" y="-38.1"/>
-<wire x1="104.14" y1="-38.1" x2="104.14" y2="-33.02" width="0.1524" layer="91"/>
-<pinref part="JP3" gate="G$1" pin="2"/>
-<wire x1="104.14" y1="-33.02" x2="114.3" y2="-33.02" width="0.1524" layer="91"/>
+<wire x1="99.06" y1="-38.1" x2="99.06" y2="-40.64" width="0.1524" layer="91"/>
+<pinref part="JP1" gate="A" pin="1"/>
+<wire x1="99.06" y1="-40.64" x2="114.3" y2="-40.64" width="0.1524" layer="91"/>
 </segment>
 </net>
@@
 </segment>
 </net>
+<net name="N$18" class="0">
+<segment>
+<pinref part="JP1" gate="A" pin="3"/>
+<wire x1="114.3" y1="-45.72" x2="96.52" y2="-45.72" width="0.1524" layer="91"/>
+<pinref part="S1" gate="G$1" pin="S"/>
+<wire x1="96.52" y1="-45.72" x2="96.52" y2="-55.88" width="0.1524" layer="91"/>
+<pinref part="C10" gate="G$1" pin="1"/>
+<wire x1="96.52" y1="-55.88" x2="96.52" y2="-63.5" width="0.1524" layer="91"/>
+<wire x1="104.14" y1="-63.5" x2="104.14" y2="-55.88" width="0.1524" layer="91"/>
+<wire x1="104.14" y1="-55.88" x2="96.52" y2="-55.88" width="0.1524" layer="91"/>
+<junction x="96.52" y="-55.88"/>
+</segment>
+</net>
